File: hardware/de10-shield/de10-shield.kicad_pcb (KiCad board)
At the start: 2 copper layers, 137.1 x 70 mm, 35 parts, among them J1 GPIO_0, J10 SW3, J11 SW4, J12 SW5, J13 SW6, J14 SW7, J15 GPIO_0_AUX, J16 GPIO_1_AUX, J17 TFT_DISPLAY, J18 LED_0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

Commit message: done
Parts:
- added H5: MountingHole_Pad, MountingHole:MountingHole_3.2mm_M3_DIN965_Pad, F.Cu at (149.0, 128.0)
- added H6: MountingHole_Pad, MountingHole:MountingHole_3.2mm_M3_DIN965_Pad, F.Cu at (155.0, 122.0)
- added J20: 5V, Connector_PinHeader_2.54mm:PinHeader_1x02_P2.54mm_Vertical, F.Cu at (146.1, 49.5)
- added J21: 3.3V, Connector_PinHeader_2.54mm:PinHeader_1x02_P2.54mm_Vertical, F.Cu at (156.2, 49.5)
- added J22: ENCODER_1, Connector_PinSocket_2.54mm:PinSocket_1x05_P2.54mm_Vertical, F.Cu at (88.0, 72.0)
- added J23: ENCODER_2, Connector_PinSocket_2.54mm:PinSocket_1x05_P2.54mm_Vertical, F.Cu at (88.0, 86.0)
- added J24: ENCODER_3, Connector_PinSocket_2.54mm:PinSocket_1x05_P2.54mm_Vertical, F.Cu at (88.0, 100.0)
- J15: value GPIO_0_AUX -> ENCODER_0; footprint Connector_PinSocket_2.54mm:PinSocket_1x20_P2.54mm_Vertical -> Connector_PinSocket_2.54mm:PinSocket_1x05_P2.54mm_Vertical
- moved C17 54.6 mm to (152.6, 110.2)
- moved TP1 54.4 mm to (155.9, 110.7)
- moved L1 54.2 mm to (147.6, 112.5), turned to 270 degrees
- moved C16 54.2 mm to (149.5, 116.4)
- moved C14 54.0 mm to (152.5, 117.0)
- moved MAX176321 54.0 mm to (152.5, 114.0)
- moved C13 54.0 mm to (156.0, 115.9)
- moved C15 54.0 mm to (155.7, 113.1)
- moved J15 49.1 mm to (88.0, 58.0), turned to 0 degrees
Connections:
- J1 pad 10: Net-(J1-Pad10) -> /DIR_0
- J1 pad 11: +5V -> Net-(J1-Pad11)
- J1 pad 12: GND -> Net-(J1-Pad12)
- J1 pad 13: /EN_0 -> Net-(J1-Pad13)
- J1 pad 15: /MS1_0 -> Net-(J1-Pad15)
- J1 pad 16: Net-(J1-Pad16) -> /I_3
- J1 pad 17: /MS2_0 -> Net-(J1-Pad17)
- J1 pad 18: Net-(J1-Pad18) -> /B_3
- J1 pad 19: /STEP_0 -> Net-(J1-Pad19)
- J1 pad 2: Net-(J1-Pad2) -> /EN_0
- J1 pad 20: Net-(J1-Pad20) -> /A_3
- J1 pad 21: /DIR_0 -> Net-(J1-Pad21)
- J1 pad 22: Net-(J1-Pad22) -> /I_2
- J1 pad 24: Net-(J1-Pad24) -> /B_2
- J1 pad 26: Net-(J1-Pad26) -> /A_2
- J1 pad 28: Net-(J1-Pad28) -> /I_1
- J1 pad 30: GND -> Net-(J1-Pad30)
- J1 pad 32: Net-(J1-Pad32) -> /B_1
- J1 pad 34: Net-(J1-Pad34) -> /A_1
- J1 pad 36: Net-(J1-Pad36) -> /I_0
- J1 pad 38: Net-(J1-Pad38) -> /B_0
- J1 pad 4: Net-(J1-Pad4) -> /MS1_0
- J1 pad 40: Net-(J1-Pad40) -> /A_0
- J1 pad 6: Net-(J1-Pad6) -> /MS2_0
- J1 pad 8: Net-(J1-Pad8) -> /STEP_0
- J15 pad 1: Net-(J1-Pad2) -> +3V3
- J15 pad 2: Net-(J1-Pad4) -> GND
- J15 pad 3: Net-(J1-Pad6) -> /A_0
- J15 pad 4: Net-(J1-Pad8) -> /B_0
- J15 pad 5: Net-(J1-Pad10) -> /I_0
- J16 pad 15: GND -> Net-(J16-Pad15)
- J16 pad 6: GND -> Net-(J16-Pad6)
- J2 pad 12: GND -> Net-(J16-Pad6)
- J2 pad 29: +3V3 -> Net-(J2-Pad29)
- J2 pad 30: GND -> Net-(J16-Pad15)
Routing:
- net VMEM: track 0.00 -> 283.9 mm, vias 0 -> 7
- net +3V3: track 0.00 -> 250.9 mm, vias 0 -> 3
- net +5V: track 0.00 -> 118.2 mm
- net GND: track 0.00 -> 106.2 mm, vias 0 -> 61
- net /DIR_0: track 0.00 -> 87.0 mm, vias 0 -> 1
- net /DIR_2: track 0.00 -> 77.7 mm
- net /LED_1: track 0.00 -> 68.3 mm, vias 0 -> 1
- net /MS2_0: track 0.00 -> 57.9 mm
- net /STEP_0: track 0.00 -> 53.5 mm, vias 0 -> 1
- net /LED_0: track 0.00 -> 52.1 mm
- net /SW5: track 0.00 -> 51.8 mm
- net /SW7: track 0.00 -> 51.7 mm
- net /EN_1: track 0.00 -> 50.1 mm, vias 0 -> 1
- net /MS1_0: track 0.00 -> 47.3 mm
- net /MS1_1: track 0.00 -> 44.1 mm, vias 0 -> 2
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- added copper zone on B.Cu, net GND
- added copper zone on F.Cu, net GND
Other:
- board size 137.1 x 70 mm -> 73 x 85 mm
- board text added: "3.3V"
- board text added: "5-36V"
- board text added: "5V"
- board text added: "A0"
- board text added: "A1"
- board text added: "A2"
- board text added: "A3"
- board text added: "B0"
- board text added: "B1"
- board text added: "B2"
- board text added: "B3"
- board text added: "BLK"
- board text added: "DC"
- board text added: "EN"
- board text added: "GND"
- board text added: "I0"
- board text added: "I1"
- board text added: "I2"
- board text added: "I3"
- board text added: "LED_0"
- board text added: "LED_1"
- board text added: "RES"
- board text added: "SCL"
- board text added: "SDA"
- board text added: "SW0"
- board text added: "SW2"
- board text added: "SW3"
- board text added: "SW4"
- board text added: "SW5"
- board text added: "SW6"
- board text added: "SW7"

Commit message: done and ordered
Parts:
- added H7: MountingHole_Pad, MountingHole:MountingHole_3.2mm_M3_DIN965_Pad, F.Cu at (118.1, 100.2)
- C13, C14: footprint Capacitor_SMD:C_0603_1608Metric -> Capacitor_SMD:C_1210_3225Metric_Pad1.33x2.70mm_HandSolder
- C15: footprint Capacitor_SMD:C_0402_1005Metric -> Capacitor_SMD:C_0603_1608Metric_Pad1.08x0.95mm_HandSolder
- C16: footprint Capacitor_SMD:C_0402_1005Metric -> Capacitor_SMD:C_0805_2012Metric_Pad1.18x1.45mm_HandSolder
- moved C16 1.50 mm to (148.0, 116.5)
- moved C14 1.30 mm to (151.8, 118.1)
- moved C15 1.29 mm to (156.6, 112.2), turned to 0 degrees
- moved TP1 1.15 mm to (156.7, 109.9)
- moved H6 1.00 mm to (155.1, 123.0)
- moved L1 0.63 mm to (147.4, 111.9)
- moved C13 0.58 mm to (156.5, 116.2)
- moved C17 0.22 mm to (152.7, 110.0), turned to 270 degrees
Routing:
- net GND: track 106.2 -> 112.7 mm, vias 61 -> 66
- net Net-(C16-Pad1): track 7.27 -> 10.9 mm
- net /STEP_0: track 53.5 -> 55.1 mm
- net Net-(C13-Pad1): track 3.51 -> 4.79 mm
- net VMEM: track 283.9 -> 284.8 mm
- net Net-(C16-Pad2): track 3.03 -> 3.92 mm
- net /MS2_3: track 34.4 -> 35.2 mm
Other:
- board size 73 x 85 mm -> 73 x 86 mm
- rule pad_to_mask_clearance: 0.051 -> 0
